File: CawDrive.kicad_sch (KiCad schematic)
At the start: 48 parts, among them CN1 XT60PW-M, J1 Conn_01x04_Pin, J2 USB_B_Micro, SW1 B3U-1000P, U1 STM32F446RETx, U2 ISO1044BDR, U3 CH340K, Y1 16MHz

Commit message: 参考MIT驱动器进行改版
Parts:
- removed C10, C7: 10uF, Capacitor_SMD:C_0603_1608Metric_Pad1.08x0.95mm_HandSolder, symbol Device:C_Small
- removed C11, C13: 0.1uF, Capacitor_SMD:C_0603_1608Metric_Pad1.08x0.95mm_HandSolder, symbol Device:C_Small
- removed C14, C16: 12pF, Capacitor_SMD:C_0603_1608Metric_Pad1.08x0.95mm_HandSolder, symbol Device:C_Small
- removed CN1: XT60PW-M, Rick_Connector:XT60PW-M, symbol Rick_Connector:XT60PW-M
- removed FPC1: XH-6PWB, Rick_Connector:XH-6PWB, symbol Rick_Connector:XH-6PWB
- removed FPC2: XH-4PWB, Rick_Connector:XH-4PWB, symbol Rick_Connector:XH-4PWB
- removed FPC3: XH-2PWB, Rick_Connector:XH-2PWB, symbol Rick_Connector:XH-2PWB
- removed J1: Conn_01x04_Pin, Connector_PinHeader_2.54mm:PinHeader_1x04_P2.54mm_Vertical, symbol Connector:Conn_01x04_Pin
- removed J2: USB_B_Micro, Rick_USB:Micro_USB_B_SMD, symbol Rick_USB:USB_B_Micro
- removed R10: 1M, Resistor_SMD:R_0603_1608Metric_Pad0.98x0.95mm_HandSolder, symbol Device:R_Small
- removed R13: 47, Resistor_SMD:R_0603_1608Metric_Pad0.98x0.95mm_HandSolder, symbol Device:R_Small
- removed R4: 0, Resistor_SMD:R_0603_1608Metric_Pad0.98x0.95mm_HandSolder, symbol Device:R_Small
- removed R7: 33, Resistor_SMD:R_0603_1608Metric_Pad0.98x0.95mm_HandSolder, symbol Device:R_Small
- removed SW1: B3U-1000P, Rick_Switch:B3U-1000P, symbol Rick_Switch:B3U-1000P
- removed TV1: SMAJ36CA/TR13, Rick_Diode:SMAJ36CA_TR13, symbol Rick_Diode:SMAJ36CA/TR13
- removed U2: ISO1044BDR, Rick_CAN:ISO1044BDR, symbol Rick_CAN:ISO1044BDR
- removed U3: CH340K, Rick_Interface_USB:CH340K, symbol Rick_Interface_USB:CH340K
- removed Y1: 16MHz, Rick_Device:Crystal_16MHz_GND24, symbol Rick_Device:Crystal_16MHz_GND24
- added H8, H9: MountingHole_Pad, CawDrive_Connector:POWER_PAD, symbol Mechanical:MountingHole_Pad
- added J1: Conn_01x11_Pin, CawDrive_Connector:SOIC-11, symbol Connector:Conn_01x11_Pin
- added J4: Conn_01x07_Pin, CawDrive_Connector:SOIC-7, symbol Connector:Conn_01x07_Pin
- added TV1: SMAJ36CA/TR13, Rick_Diode:SMAJ36CA_TR13_SMA(DO-214AC), symbol Rick_Diode:SMAJ36CA/TR13
- added U2: NCV7342MW3R2G, Rick_CAN:NCV7342MW3R2G_DFN-8_L3.0-W3.0-P0.65-BL-EP, symbol Rick_CAN:NCV7342MW3R2G
- added X1: Crystal_16MHz_15pF_3P, Rick_Crystal:Crystal_SMD3213-3P, symbol Rick_Device:Crystal_16MHz_15pF_3P
- C1, C12, C2, C3, C4, C5, C6, C9: footprint Capacitor_SMD:C_0603_1608Metric_Pad1.08x0.95mm_HandSolder -> Capacitor_SMD:C_0402_1005Metric_Pad0.74x0.62mm_HandSolder
- C14: renamed from C15; footprint Capacitor_SMD:C_0603_1608Metric_Pad1.08x0.95mm_HandSolder -> Capacitor_SMD:C_0402_1005Metric_Pad0.74x0.62mm_HandSolder
- C8: value 100nF -> 0.1uF; footprint Capacitor_SMD:C_0603_1608Metric_Pad1.08x0.95mm_HandSolder -> Capacitor_SMD:C_0402_1005Metric_Pad0.74x0.62mm_HandSolder
- D1: footprint LED_SMD:LED_0603_1608Metric_Pad1.05x0.95mm_HandSolder -> LED_SMD:LED_0402_1005Metric_Pad0.77x0.64mm_HandSolder
- D2: value DRV_A_STA_LED -> DRV_STA_LED; footprint LED_SMD:LED_0603_1608Metric_Pad1.05x0.95mm_HandSolder -> LED_SMD:LED_0402_1005Metric_Pad0.77x0.64mm_HandSolder
- H1, H2, H3, H4: footprint MountingHole:MountingHole_3.5mm_Pad_Via -> MountingHole:MountingHole_2.5mm_Pad_Via
- L1: footprint Inductor_SMD:L_0603_1608Metric_Pad1.05x0.95mm_HandSolder -> Inductor_SMD:L_0402_1005Metric_Pad0.77x0.64mm_HandSolder
- R1, R2, R3, R5, R6, R8, R9: footprint Resistor_SMD:R_0603_1608Metric_Pad0.98x0.95mm_HandSolder -> Resistor_SMD:R_0402_1005Metric_Pad0.72x0.64mm_HandSolder
- R10: renamed from R11; footprint Resistor_SMD:R_0603_1608Metric_Pad0.98x0.95mm_HandSolder -> Resistor_SMD:R_0402_1005Metric_Pad0.72x0.64mm_HandSolder
- R11: renamed from R12; footprint Resistor_SMD:R_0603_1608Metric_Pad0.98x0.95mm_HandSolder -> Resistor_SMD:R_0402_1005Metric_Pad0.72x0.64mm_HandSolder
Connections:
- net I2C1_SCL is gone; now on net CAN_TX: U1.58 (PB6)
- net +3.3V: now also R5.2, J1.1 (Pin_1), J1.6 (Pin_6), J4.1 (Pin_1), U2.5 (VIO); no longer R5.1
- net +36V: now also H9.1, TV1.1 (K)
- net +5V: now also C12.2, U2.3 (VCC); no longer C12.1
- net CAN_N: now also J4.7 (Pin_7), U2.6 (CANL)
- net CAN_P: now also J4.6 (Pin_6), U2.7 (CANH)
- net DRV_CAL: now also U1.38 (PC7); no longer U1.40 (PC9)
- net DRV_FAULT: now also U1.40 (PC9); no longer U1.38 (PC7)
- net GND: now also C12.1, H8.1, J1.2 (Pin_2), J1.7 (Pin_7), J4.2 (Pin_2), J4.5 (Pin_5), TV1.2 (A), U2.2 (GND), X1.2 (GND); no longer C12.2, H1.1, H2.1
- net HSE_IN: now also X1.1 (OSC1)
- net HSE_OUT: now also X1.3 (OSC2)
- net MCU_STA: now also U1.54 (PD2); no longer U1.2 (PC13)
- net RESET: now also J1.3 (Pin_3)
- net SPI1_MISO: now also U1.22 (PA6), J1.10 (Pin_10); no longer U1.56 (PB4)
- net SPI1_MOSI: now also U1.23 (PA7), J1.11 (Pin_11); no longer U1.57 (PB5)
- net SPI1_NSS: now also U1.20 (PA4), J1.8 (Pin_8); no longer U1.54 (PD2)
- net SPI1_SCK: now also U1.21 (PA5), J1.9 (Pin_9); no longer U1.55 (PB3)
- net SWCLK: now also J1.5 (Pin_5)
- net SWDIO: now also R5.1, J1.4 (Pin_4); no longer R5.2
- net USART2_TX: now reaches U1.16 (PA2)
- net USART2_TX: now also J4.4 (Pin_4)
- net USART2_RX: now reaches U1.17 (PA3)
- net USART2_RX: now also J4.3 (Pin_3)
- net ADC1_IN8: now reaches U1.26 (PB0)
- net ADC1_IN9: now reaches U1.27 (PB1)
- net TIM1_BKIN: now reaches U1.33 (PB12)
- net TIM1_BKIN: now also U1.37 (PC6)
- net ADC1_IN0: no longer names the net of U1.14 (PA0)
- net ADC1_IN1: no longer names the net of U1.15 (PA1)
- net CAN1_RX renamed CAN_RX
- net CAN_RX: now also U1.57 (PB5), U2.4 (RxD)
- net CAN1_TX renamed CAN_TX
- net CAN_TX: now also U2.1 (TxD)
- net CH340_RXD: no longer names the net of U1.29 (PB10)
- net CH340_TXD: no longer names the net of U1.25 (PC5)
- net DRV_A_STA: no longer names the net of U1.3 (PC14)
- net DRV_A_STA: no longer R11.2
- net GND1: no longer names the net of H4.1
- net GND1: no longer H3.1
- net I2C1_SDA: no longer names the net of U1.59 (PB7)
- new net CAN_STB: U1.56 (PB4), U2.8 (STB)
- new net DRV_STA: R11.2, U1.55 (PB3)
- no-connect marks 24 -> 19
Other:
- note removed: "I2C接口"
- note removed: "SPI接口"
- note removed: "SWD调试接口"
- note removed: "USB串口"
- moved on the sheet: C1, C12, C14, C9, R1, R10, R2, R3, R5, R6, R8, U1

Commit message: 将线性稳压芯片和CAN芯片替换成TI的相关型号
Parts:
- removed U2: NCV7342MW3R2G, Rick_CAN:NCV7342MW3R2G_DFN-8_L3.0-W3.0-P0.65-BL-EP, symbol Rick_CAN:NCV7342MW3R2G
- added U3: TCAN1044DRBRQ1, Rick_CAN:TCAN1044DRBRQ1_DFN-8_L3.0-W3.0-P0.65-TL-EP2.4, symbol Rick_CAN:TCAN1044DRBRQ1
Connections:
- net +3.3V: now also U3.5 (NC/VIO)
- net +5V: now also U3.3 (VCC)
- net CAN_N: now also U3.6 (CANL)
- net CAN_P: now also U3.7 (CANH)
- net CAN_RX: now also U3.4 (RXD)
- net CAN_STB: now also U3.8 (STB)
- net CAN_TX: now also U3.1 (TXD)
- net GND: now also U3.2 (GND), U3.9 (EP)
Other:
- note added: "接口"
- moved on the sheet: C9, J1, J4, R8

Commit message: 优化布线
Parts:
- added D4: PWR_STA_LED, LED_SMD:LED_0402_1005Metric_Pad0.77x0.64mm_HandSolder, symbol Device:LED_Small
- added R4: 0Ω, Resistor_SMD:R_0402_1005Metric_Pad0.72x0.64mm_HandSolder, symbol Device:R_Small
- added R7: 510, Resistor_SMD:R_0402_1005Metric_Pad0.72x0.64mm_HandSolder, symbol Device:R_Small
- R2: value 0 -> 0Ω
Connections:
- net +3.3V: now also D4.2 (A)
- net GND: now also R4.2, R7.2; no longer H8.1, TV1.2 (A)
- new net: D4.1 (K), R7.1
- new net GND1: H8.1, R4.1, TV1.2 (A)
Changed lines of the file:
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@@
+    (stroke (width 0) (type default))
+  )
+  (wire (pts (xy 102.87 24.13) (xy 105.41 24.13))
     (stroke (width 0) (type default))
   )
@@
     (stroke (width 0) (type default))
   )
+  (wire (pts (xy 110.49 24.13) (xy 113.03 24.13))
+    (stroke (width 0) (type default))
+  )
   (wire (pts (xy 153.67 35.56) (xy 160.02 35.56))
     (stroke (width 0) (type default))
@@
     (stroke (width 0) (type default))
   )
-  (wire (pts (xy 102.87 24.13) (xy 113.03 24.13))
-    (stroke (width 0) (type default))
-  )
   (wire (pts (xy 226.06 94.615) (xy 228.6 94.615))
     (stroke (width 0) (type default))
@@
     (stroke (width 0) (type default))
   )
+  (wire (pts (xy 261.62 40.005) (xy 261.62 40.64))
+    (stroke (width 0) (type default))
+  )
   (wire (pts (xy 227.33 46.99) (xy 238.76 46.99))
     (stroke (width 0) (type default))
@@
     (stroke (width 0) (type default))
   )
+  (wire (pts (xy 261.62 51.435) (xy 261.62 52.07))
+    (stroke (width 0) (type default))
+  )
   (wire (pts (xy 68.58 29.21) (xy 68.58 30.48))
     (stroke (width 0) (type default))
@@
   )
   (wire (pts (xy 233.68 149.86) (xy 222.25 149.86))
+    (stroke (width 0) (type default))
+  )
+  (wire (pts (xy 261.62 45.72) (xy 261.62 46.355))
     (stroke (width 0) (type default))
   )
@@
     (fill (type none))
   )
-  (rectangle (start 254 54.61) (end 283.21 88.9)
+  (rectangle (start 254 33.02) (end 283.21 88.9)
     (stroke (width 0) (type dash))
     (fill (type none))
@@
     )
   )
+  (symbol (lib_id "Device:LED_Small") (at 261.62 43.18 90) (unit 1)
+    (in_bom yes) (on_board yes) (dnp no)
+    (property "Reference" "D4" (at 262.89 41.91 90)
+      (effects (font (size 1.27 1.27)) (justify right))
+    )
+    (property "Value" "PWR_STA_LED" (at 257.81 36.83 0)
+      (effects (font (size 1.27 1.27)) (justify right))
+    )
+    (property "Footprint" "LED_SMD:LED_0402_1005Metric_Pad0.77x0.64mm_HandSolder" (at 261.62 43.18 90)
+      (effects (font (size 1.27 1.27)) hide)
+    )
+    (property "Datasheet" "~" (at 261.62 43.18 90)
+      (effects (font (size 1.27 1.27)) hide)
+    )
+    (pin "1")
+    (pin "2")
+    (instances
+      (project "CawDrive"
+        (path "/80524a83-b783-469c-b956-da06086e2ffd"
+          (reference "D4") (unit 1)
+        )
+      )
+    )
+  )
   (symbol (lib_id "power:GND") (at 38.1 76.2 0) (unit 1)
     (in_bom yes) (on_board yes) (dnp no)
@@
     )
   )
+  (symbol (lib_id "Device:R_Small") (at 107.95 24.13 90) (unit 1)
+    (in_bom yes) (on_board yes) (dnp no) (fields_autoplaced)
+    (property "Reference" "R4" (at 107.95 19.05 90)
+      (effects (font (size 1.27 1.27)))
+    )
+    (property "Value" "0Ω" (at 107.95 21.59 90)
+      (effects (font (size 1.27 1.27)))
+    )
+    (property "Footprint" "Resistor_SMD:R_0402_1005Metric_Pad0.72x0.64mm_HandSolder" (at 107.95 24.13 0)
+      (effects (font (size 1.27 1.27)) hide)
+    )
+    (property "Datasheet" "~" (at 107.95 24.13 0)
+      (effects (font (size 1.27 1.27)) hide)
+    )
+    (pin "1")
+    (pin "2")
+    (instances
+      (project "CawDrive"
+        (path "/80524a83-b783-469c-b956-da06086e2ffd"
+          (reference "R4") (unit 1)
+        )
+      )
+    )
+  )
   (symbol (lib_id "Device:C_Small") (at 78.74 26.67 0) (unit 1)
     (in_bom yes) (on_board yes) (dnp no)
@@
         (path "/80524a83-b783-469c-b956-da06086e2ffd"
           (reference "#PWR016") (unit 1)
+        )
+      )
+    )
+  )
+  (symbol (lib_id "power:GND") (at 261.62 52.07 0) (unit 1)
+    (in_bom yes) (on_board yes) (dnp no)
+    (property "Reference" "#PWR044" (at 261.62 58.42 0)
+      (effects (font (size 1.27 1.27)) hide)
+    )
+    (property "Value" "GND" (at 265.43 53.975 0)
+      (effects (font (size 1.27 1.27)))
+    )
+    (property "Footprint" "" (at 261.62 52.07 0)
+      (effects (font (size 1.27 1.27)) hide)
+    )
+    (property "Datasheet" "" (at 261.62 52.07 0)
+      (effects (font (size 1.27 1.27)) hide)
+    )
+    (pin "1")
+    (instances
+      (project "CawDrive"
+        (path "/80524a83-b783-469c-b956-da06086e2ffd"
+          (reference "#PWR044") (unit 1)
         )
       )
@@
     )
   )
+  (symbol (lib_id "power:+3.3V") (at 261.62 40.005 0) (unit 1)
+    (in_bom yes) (on_board yes) (dnp no)
+    (property "Reference" "#PWR035" (at 261.62 43.815 0)
+      (effects (font (size 1.27 1.27)) hide)
+    )
+    (property "Value" "+3.3V" (at 261.62 36.195 0)
+      (effects (font (size 1.27 1.27)))
+    )
+    (property "Footprint" "" (at 261.62 40.005 0)
+      (effects (font (size 1.27 1.27)) hide)
+    )
+    (property "Datasheet" "" (at 261.62 40.005 0)
+      (effects (font (size 1.27 1.27)) hide)
+    )
+    (pin "1")
+    (instances
+      (project "CawDrive"
+        (path "/80524a83-b783-469c-b956-da06086e2ffd"
+          (reference "#PWR035") (unit 1)
+        )
+      )
+    )
+  )
   (symbol (lib_id "power:+3.3V") (at 139.7 31.75 0) (unit 1)
     (in_bom yes) (on_board yes) (dnp no) (fields_autoplaced)
@@
         (path "/80524a83-b783-469c-b956-da06086e2ffd"
           (reference "R1") (unit 1)
+        )
+      )
+    )
+  )
+  (symbol (lib_id "Device:R_Small") (at 261.62 48.895 0) (unit 1)
+    (in_bom yes) (on_board yes) (dnp no) (fields_autoplaced)
+    (property "Reference" "R7" (at 264.16 47.625 0)
+      (effects (font (size 1.27 1.27)) (justify left))
+    )
+    (property "Value" "510" (at 264.16 50.165 0)
+      (effects (font (size 1.27 1.27)) (justify left))
+    )
+    (property "Footprint" "Resistor_SMD:R_0402_1005Metric_Pad0.72x0.64mm_HandSolder" (at 261.62 48.895 0)
+      (effects (font (size 1.27 1.27)) hide)
+    )
+    (property "Datasheet" "~" (at 261.62 48.895 0)
+      (effects (font (size 1.27 1.27)) hide)
+    )
+    (pin "1")
+    (pin "2")
+    (instances
+      (project "CawDrive"
+        (path "/80524a83-b783-469c-b956-da06086e2ffd"
+          (reference "R7") (unit 1)
         )
       )
@@
       (effects (font (size 1.27 1.27)) (justify left))
     )
-    (property "Value" "0" (at 79.375 157.48 90)
+    (property "Value" "0Ω" (at 80.645 157.48 90)
       (effects (font (size 1.27 1.27)) (justify left))
     )
@@
       (effects (font (size 1.27 1.27)) hide)
     )
+    (property "无标题字段" "" (at 79.375 157.48 0)
+      (effects (font (size 1.27 1.27)) hide)
+    )

Commit message: 升级主控STM32G474，增加AS5047P编码器，支持NTC温度采样
Parts:
- removed J1: Conn_01x11_Pin, CawDrive_Connector:SOIC-11, symbol Connector:Conn_01x11_Pin
- removed J4: Conn_01x07_Pin, CawDrive_Connector:SOIC-7, symbol Connector:Conn_01x07_Pin
- removed R3, R5, R6: 10k, Resistor_SMD:R_0402_1005Metric_Pad0.72x0.64mm_HandSolder, symbol Device:R_Small
- removed U1: STM32F446RETx, Package_QFP:LQFP-64_10x10mm_P0.5mm, symbol MCU_ST_STM32F4:STM32F446RETx
- added C11, C17: 0.1uF, Capacitor_SMD:C_0402_1005Metric_Pad0.74x0.62mm_HandSolder, symbol Device:C_Small
- added CN1, CN2: WAFER-SH1.0-6PWB, Rick_Connector:CONN-SMD_6P-P1.00_XUNPU_WAFER-SH1.0-6PWB, symbol Rick_Connector:WAFER-SH1.0-6PWB
- added R12: 10K, Resistor_SMD:R_0402_1005Metric_Pad0.72x0.64mm_HandSolder, symbol Device:R_Small
- added R15: 0Ω, Resistor_SMD:R_0402_1005Metric_Pad0.72x0.64mm_HandSolder, symbol Device:R_Small
- added R20, R21: 10k, Resistor_SMD:R_0402_1005Metric_Pad0.72x0.64mm_HandSolder, symbol Device:R_Small
- added U1: AS5047P-ATSM, Rick_Sensor:AS5047P-ATSM, symbol Rick_Sensor:AS5047P-ATSM
- added U4: STM32G474RETx, Package_QFP:LQFP-64_10x10mm_P0.5mm, symbol MCU_ST_STM32G4:STM32G474RETx
- added U5, U6: WAFER-SH1.0-2PWB, Rick_Connector:CONN-SMD_2P-P1.00_XUNPU_WAFER-SH1.0-2PWB, symbol Rick_Connector:WAFER-SH1.0-2PWB
- C1: value 2.2uF -> 0.1uF
- H1, H2, H3, H4, H8, H9: now not fitted
- R1: value 10K -> 10k
- R11, R7, R9: value 510 -> 510Ω
- R2: value 0Ω -> 10k
- R8: value 120 -> 120Ω 1%
- X1: value Crystal_16MHz_15pF_3P -> CSTNE16M0V530000R0
Connections:
- net +3.3V: now also R1.2, R2.1, C17.2, CN1.6, CN2.4, R20.2, U1.11 (VDD), U1.12 (VDD3V3), U4.1 (VBAT), U4.16 (VDD), U4.32 (VDD), U4.48 (VDD), U4.64 (VDD)
- net +3.3VA: now also C11.1, U4.28 (VREF+), U4.29 (VDDA)
- net CAN_N: now also U5.1
- net CAN_P: now also U5.2
- net DRV_CAL: now also U4.39 (PC7)
- net DRV_ENABLE: now also U4.40 (PC8)
- net DRV_FAULT: now also U4.41 (PC9)
- net DRV_STA: now also U4.25 (PB1)
- net GND: now also C1.1, C11.2, C17.1, CN1.5, CN2.3, R12.2, R15.2, R21.2, U1.13 (GND), U1.5 (Test), U4.15 (VSS), U4.31 (VSS), U4.47 (VSS), U4.63 (VSS), U6.2; no longer C1.2, R1.1, R2.2
- net HSE_IN: now also U4.5 (PF0)
- net HSE_OUT: now also U4.6 (PF1)
- net MCU_STA: now also U4.26 (PB2)
- net RESET: now also U4.7 (PG10)
- net SPI1_MISO: now also R2.2, CN1.3, U4.20 (PA6)
- net SPI1_MOSI: now also CN1.2, U4.21 (PA7)
- net SPI1_NSS: now also CN1.1, U4.18 (PA4)
- net SPI1_SCK: now also CN1.4, U4.19 (PA5)
- net SPI3_MISO: now also U1.3 (MISO), U4.53 (PC11)
- net SPI3_MOSI: now also U1.4 (MOSI), U4.54 (PC12)
- net SPI3_SCK: now also U1.2 (CLK), U4.52 (PC10)
- net SWCLK: now also CN2.1, R21.1, U4.50 (PA14)
- net SWDIO: now also CN2.2, R20.1, U4.49 (PA13)
- net TIM1_BKIN: now also U4.34 (PB12), U4.38 (PC6)
- net CAN_RX renamed FDCAN_RX
- net FDCAN_RX: now also U4.56 (PB3), U4.58 (PB5)
- net CAN_STB renamed FDCAN_STB
- net FDCAN_STB: now also U4.55 (PD2)
- net CAN_TX renamed FDCAN_TX
- net FDCAN_TX: now also U4.57 (PB4), U4.59 (PB6)
- new net: R12.1, U4.61 (PB8)
- new net: R15.1, U4.27 (VSSA)
- new net ADC1_IN1: U4.12 (PA0)
- new net ADC1_IN2: U4.13 (PA1)
- new net ADC1_IN3: C1.2, R1.1, U4.14 (PA2), U6.1
- new net AS5047P_NSS: U1.1 (CSn), U4.46 (PA12)
- new net DRV_SPI_NSS: U4.51 (PA15)
- new net TIM1_CH1: U4.42 (PA8)
- new net TIM1_CH1N: U4.35 (PB13)
- new net TIM1_CH2: U4.43 (PA9)
- new net TIM1_CH2N: U4.36 (PB14)
- new net TIM1_CH3: U4.44 (PA10)
- new net TIM1_CH3N: U4.37 (PB15)
- new net USART1_RX: CN2.6, U4.23 (PC5)
- new net USART1_TX: CN2.5, U4.22 (PC4)
- no-connect marks 19 -> 32
Other:
- note added: "位置传感器"
- note added: "温度采样"
- moved on the sheet: C12, C14, C9, D4, R10, R7, R8, U3
