File: PCB/CawDrive.kicad_pcb (KiCad board)
At the start: 4 copper layers, 50 x 42 mm, 108 parts, among them CN2 WAFER-SH1.0-6PWB, CN3 WAFER-SH1.0-4PWB, Q10 TPH3R704PL, Q11 TPH3R704PL, Q12 TPH3R704PL, Q7 TPH3R704PL, Q8 TPH3R704PL, Q9 TPH3R704PL, U1 TJA1051T/3/1J, U10 WAFER-SH1.0-2PWB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

Commit message: 优化布线，生成Gerber文件
Parts:
- added kibuzzard-67F4292F: G***, kibuzzard-67F4292F, B.Cu at (157.5, 82.4)
- C19: value 33nF -> 0.1uF/50V
- R1, R20: value 10k -> 10k 1%
- R12: value 3k -> 3k 1%
- R18, R19, R22: value 1mΩ 1% -> 5mΩ 1%
- R21: value 10k -> NTC
- R8: value 75k -> 75k 1%
Routing:
- net GND: track 80.7 -> 90.4 mm
- net /TIM1_CH2: track 23.8 -> 22.1 mm
- net /ADC1_IN0: track 24.3 -> 23.0 mm
- net /DRV_STA: track 15.4 -> 16.6 mm
- net /TIM1_BKIN: track 7.37 -> 8.45 mm
- net /SPI1_SCK: track 9.82 -> 10.8 mm
- net /TIM1_CH3: track 26.2 -> 27.1 mm
- net /DRV_SPI_NSS: track 18.4 -> 19.3 mm
- net /TIM1_CH1: track 19.0 -> 18.1 mm
- net /SPI3_MOSI: track 22.2 -> 23.0 mm
- net /SPI1_MOSI: track 9.19 -> 9.93 mm
- net /TIM1_CH3N: track 29.0 -> 29.7 mm
- net /SWCLK: track 26.2 -> 25.5 mm
- net /ADC2_IN1: track 25.1 -> 24.5 mm
- net /ADC3_IN2: track 24.8 -> 25.5 mm
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